Commit message: add imu_link in urdf, add imu_broadcaster in config folder, add start imu_broadcaster controller in launch real robot file. Finally enale show log data from MPU6050

File: my_robot_description/urdf/lidar.xacro (robot description, xacro)
@@ -10,4 +10,5 @@
             <geometry>
                 <cylinder radius="${wheel_radius}" length="${wheel_length}" />
+                <!-- <mesh filename="package://my_robot_description/meshes/lidar_link.stl" scale="0.001 0.001 0.001"/> -->
             </geometry>
             <origin xyz="0 0 0" rpy="0 0 0" />
@@ -23,31 +24,33 @@
                                         xyz="0 0 0" rpy="0 0 0" />
     </link>
-   <gazebo reference="laser_frame">
-        <material>Gazebo/Red</material>
-        <sensor name="laser" type="ray">
-            <pose> 0 0 0 0 0 0 </pose>
-            <visualize>true</visualize>
-            <update_rate>10</update_rate>
-            <ray>
-                <scan>
-                    <horizontal>
-                        <samples>360</samples>
-                        <min_angle>-3.14</min_angle>
-                        <max_angle>3.14</max_angle>
-                    </horizontal>
-                </scan>
-                <range>
-                    <min>0.3</min>
-                    <max>12</max>
-                </range>
-            </ray>
-            <plugin name="laser_controller" filename="libgazebo_ros_ray_sensor.so">
-                <ros>
-                    <remapping>~/out:=scan</remapping>
-                </ros>
-                <output_type>sensor_msgs/LaserScan</output_type>
-                <frame_name>laser_frame</frame_name>
-            </plugin>
-        </sensor>
-    </gazebo>
+    <xacro:if value="$(arg use_ros2_control)">
+        <gazebo reference="laser_frame">
+                <material>Gazebo/Red</material>
+                <sensor name="laser" type="ray">
+                    <pose> 0 0 0 0 0 0 </pose>
+                    <visualize>true</visualize>
+                    <update_rate>10</update_rate>
+                    <ray>
+                        <scan>
+                            <horizontal>
+                                <samples>360</samples>
+                                <min_angle>-3.14</min_angle>
+                                <max_angle>3.14</max_angle>
+                            </horizontal>
+                        </scan>
+                        <range>
+                            <min>0.3</min>
+                            <max>12</max>
+                        </range>
+                    </ray>
+                    <plugin name="laser_controller" filename="libgazebo_ros_ray_sensor.so">
+                        <ros>
+                            <remapping>~/out:=scan</remapping>
+                        </ros>
+                        <output_type>sensor_msgs/LaserScan</output_type>
+                        <frame_name>laser_frame</frame_name>
+                    </plugin>
+                </sensor>
+            </gazebo>
+    </xacro:if>
 </robot>

File: my_robot_description/urdf/mobile_base.xacro (robot description, xacro)
@@ -1,4 +1,5 @@
 <?xml version="1.0"?>
 <robot xmlns:xacro="http://www.ros.org/wiki/xacro">
+    <!-- declare detail properties of diff bot -->
     <xacro:property name="base_length" value="0.6" />
     <xacro:property name="base_width" value="0.4" />
@@ -6,4 +7,5 @@
     <xacro:property name="wheel_radius" value="0.1" />
     <xacro:property name="wheel_length" value="0.05" />
+    <!-- declare link of diff bot -->
     <link name="base_footprint" />
     <link name="base_link">
@@ -96,4 +98,21 @@
                            xyz="0 0 0" rpy="0 0 0" />
     </link>
+    <link name="imu_link">
+        <visual>
+            <origin xyz="0.0 0.0 0.0" rpy="0.0 0.0 0.0"/>
+            <geometry>
+                <!-- <mesh filename="package://my_robot_description/meshes/imu_link.stl"/>          -->
+                <box size="0.0208 0.0158 0.0016"/>
+            </geometry>
+        </visual>
+        <collision>
+            <origin xyz="0.0 0.0 0.0" rpy="0.0 0.0 0.0"/>
+            <geometry>
+                <!-- <mesh filename="package://my_robot_description/meshes/imu_link.stl"/>          -->
+            <box size="0.0208 0.0158 0.0016"/>
+            </geometry>
+        </collision>
+    </link>
+    <!-- declare joint of diff bot -->
     <joint name="base_joint" type="fixed">
         <parent link="base_footprint" />
@@ -128,3 +147,8 @@
         <origin xyz="${-base_length/4} 0.0 ${1.5*base_height}" rpy="0.0 0.0 0.0"/>
     </joint>
+    <joint name="imu_joint" type="fixed">
+        <parent link="base_link"/>
+        <child link="imu_link"/>
+        <origin xyz="${-base_length*0.3976} ${-base_width*0.3533} ${base_height + 0.0233}" rpy="0.0 0.0 0.0"/>
+    </joint>
 </robot>

File: my_robot_description/urdf/ros2_control_gazebo.xacro (robot description, xacro)
@@ -3,4 +3,5 @@
     <!-- use real ros2_control -->
     <xacro:unless value="$(arg sim_mode)">
+        <!-- stm32 serial -->
         <ros2_control name="HardwareMotor" type="system">
             <hardware>
@@ -25,4 +26,24 @@
             </joint>
         </ros2_control>
+        <!-- MPU6050 sensor not use in PC-->
+        <ros2_control name='MPU6050' type='sensor'>
+            <hardware>
+              <plugin>mpu6050/MPU6050Hardware</plugin>
+                <param name='sensor_name'>mpu6050</param>
+                <param name='frame_id'>imu_link</param>
+            </hardware>
+            <sensor name='mpu6050'>
+              <state_interface name='orientation.x'/>
+              <state_interface name='orientation.y'/>
+              <state_interface name='orientation.z'/>
+              <state_interface name='orientation.w'/>
+              <state_interface name='angular_velocity.x'/>
+              <state_interface name='angular_velocity.y'/>
+              <state_interface name='angular_velocity.z'/>
+              <state_interface name='linear_acceleration.x'/>
+              <state_interface name='linear_acceleration.y'/>
+              <state_interface name='linear_acceleration.z'/>
+            </sensor>
+          </ros2_control>
     </xacro:unless>
     <!-- use simulate ros2 control -->
