Commit message: update code of mpu6050 driver so that can run on pi and enable show log data from pmu 6050

File: my_robot_description/urdf/mobile_base.xacro (robot description, xacro)
@@ -150,5 +150,5 @@
         <parent link="base_link"/>
         <child link="imu_link"/>
-        <origin xyz="${-base_length*0.3976} ${-base_width*0.3533} ${base_height + 0.0233}" rpy="0.0 0.0 0.0"/>
+        <origin xyz="${-base_length*0.3976} ${-base_width*0.3533} ${base_height + 0.0233}" rpy="0.0 0.0 ${-pi/2}"/>
     </joint>
 </robot>

File: my_robot_description/urdf/ros2_control_gazebo.xacro (robot description, xacro)
@@ -29,5 +29,5 @@
         <ros2_control name='MPU6050' type='sensor'>
             <hardware>
-              <plugin>mpu6050/MPU6050Hardware</plugin>
+              <plugin>mpu6050_driver/MPU6050Hardware</plugin>
                 <param name='sensor_name'>mpu6050</param>
                 <param name='frame_id'>imu_link</param>
