Commit message: disable to receive data from MPU6050, because it lead to wrong fusion and change orientation of imu in urdf, recreate frame data between ros2 and stm32

File: my_robot_description/urdf/mobile_base_v1.xacro (robot description, xacro)
@@ -156,5 +156,5 @@
         <parent link="base_link"/>
         <child link="imu_link"/>
-        <origin xyz="${imu_x} ${-imu_y} ${imu_z}" rpy="0.0 0.0 ${-pi/2}"/>
+        <origin xyz="${imu_x} ${-imu_y} ${imu_z}" rpy="0.0 0.0 0.0"/>
     </joint>
 </robot>

File: my_robot_description/urdf/ros2_control_gazebo.xacro (robot description, xacro)
@@ -7,5 +7,5 @@
             <hardware>
                 <plugin>diffbot_system/DiffbotInterface</plugin>
-                <param name="port">//dev/serial/by-path/platform-fd500000.pcie-pci-0000:01:00.0-usb-0:1.2:1.0-port0</param>
+                <param name="port">/dev/serial/by-path/platform-fd500000.pcie-pci-0000:01:00.0-usb-0:1.2:1.0-port0</param>
             </hardware>
             <joint name="base_right_wheel_joint">
