Commit message: can run robot successfully with encoder odom + lidar scan without SLAM (no IMU and fusion between enc + IMU)

File: my_robot_description/urdf/mobile_base_v2.xacro (robot description, xacro)
@@ -157,5 +157,5 @@
         <parent link="base_link"/>
         <child link="imu_link"/>
-        <origin xyz="${imu_x - base_length/2} ${-imu_y} ${imu_z}" rpy="0.0 0.0 ${-pi/2}"/>
+        <origin xyz="${imu_x - base_length/2} ${-imu_y} ${imu_z}" rpy="0.0 0.0 0.0"/>
     </joint>
 </robot>

File: my_robot_description/urdf/ros2_control_gazebo.xacro (robot description, xacro)
@@ -27,5 +27,5 @@
         </ros2_control>
         <!-- MPU6050 sensor not use in PC-->
-        <ros2_control name='MPU6050' type='sensor'>
+        <!-- <ros2_control name='MPU6050' type='sensor'>
             <hardware>
               <plugin>mpu6050_driver/MPU6050Hardware</plugin>
@@ -45,5 +45,5 @@
               <state_interface name='linear_acceleration.z'/>
             </sensor>
-          </ros2_control>
+          </ros2_control> -->
     </xacro:unless>
     <!-- use simulate ros2 control -->
